File: Urban Battery - BMS_complement.kicad_sch (KiCad schematic)
At the start: 38 parts, among them J1 BMS IO, J10 E-Stop, J11 Contactor Connector, J12 Thermistor, J13 Thermistor, J14 Thermistor, J2 OLED Header, J3 CAN Connector, J4 CAN Connector, J5 Charge Connector, J6 Battery Connector, J7 E-Stop, J8 E-Stop, J9 E-Stop, K1 Charge_Relay, K2 Contactor_Relay, SW1 SW_SPST, SW2 SW_DPDT_x2, SW3 CAN_TERM, U1 MCP2515-xSO, U2 MCP2551-I-SN, U3 LM2575HVS-12/NOPB, Y1 8MHz

Commit message: switched 12V charge and contactor relays for 48V relays, updated symbol and footprint accordingly
Parts:
- K1, K2: footprint Relay_THT:Relay_1P1T_NO_10x24x18.8mm_Panasonic_ADW11xxxxW_THT -> Relay_THT:Relay_SPST_Schrack-RT1-16A-FormA_RM5mm
Changed lines of the file:
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@@
       (effects (font (size 1.27 1.27)) (justify left))
     )
-    (property "Footprint" "Relay_THT:Relay_1P1T_NO_10x24x18.8mm_Panasonic_ADW11xxxxW_THT" (id 2) (at 248.285 69.85 0)
-      (effects (font (size 1.27 1.27)) hide)
-    )
-    (property "Datasheet" "https://www.panasonic-electric-works.com/pew/es/downloads/ds_dw_hl_en.pdf" (id 3) (at 214.63 68.58 0)
+    (property "Footprint" "Relay_THT:Relay_SPST_Schrack-RT1-16A-FormA_RM5mm" (id 2) (at 248.285 69.85 0)
+      (effects (font (size 1.27 1.27)) hide)
+    )
+    (property "Datasheet" "https://www.te.com/commerce/DocumentDelivery/DDEController?Action=srchrtrv&DocNm=RT1&DocType=DS&DocLang=English" (id 3) (at 214.63 68.58 0)
       (effects (font (size 1.27 1.27)) hide)
     )
@@
       (effects (font (size 1.27 1.27)) (justify left))
     )
-    (property "Footprint" "Relay_THT:Relay_1P1T_NO_10x24x18.8mm_Panasonic_ADW11xxxxW_THT" (id 2) (at 253.365 132.08 0)
-      (effects (font (size 1.27 1.27)) hide)
-    )
-    (property "Datasheet" "https://www.panasonic-electric-works.com/pew/es/downloads/ds_dw_hl_en.pdf" (id 3) (at 219.71 130.81 0)
+    (property "Footprint" "Relay_THT:Relay_SPST_Schrack-RT1-16A-FormA_RM5mm" (id 2) (at 253.365 132.08 0)
+      (effects (font (size 1.27 1.27)) hide)
+    )
+    (property "Datasheet" "https://www.te.com/commerce/DocumentDelivery/DDEController?Action=srchrtrv&DocNm=RT1&DocType=DS&DocLang=English" (id 3) (at 219.71 130.81 0)
       (effects (font (size 1.27 1.27)) hide)
     )
@@
     )
     (path "/950489a6-5e74-426b-bb53-89098511df09"
-      (reference "K1") (unit 1) (value "Charge_Relay") (footprint "Relay_THT:Relay_1P1T_NO_10x24x18.8mm_Panasonic_ADW11xxxxW_THT")
+      (reference "K1") (unit 1) (value "Charge_Relay") (footprint "Relay_THT:Relay_SPST_Schrack-RT1-16A-FormA_RM5mm")
     )
     (path "/ea90f9ac-3a1c-4bd6-87e3-9c84b8c1984a"
-      (reference "K2") (unit 1) (value "Contactor_Relay") (footprint "Relay_THT:Relay_1P1T_NO_10x24x18.8mm_Panasonic_ADW11xxxxW_THT")
+      (reference "K2") (unit 1) (value "Contactor_Relay") (footprint "Relay_THT:Relay_SPST_Schrack-RT1-16A-FormA_RM5mm")
     )
     (path "/cd4715e8-d7f5-41c0-9b30-f49dea5c4913"
